Commit message: camera added

File: bal_robot_urdf_description/urdf/bal_robot_urdf.xacro (robot description, xacro)
@@ -53,5 +53,5 @@
   </inertial>
   <visual>
-    <origin xyz="-0.187737 -0.001226 -0.082264" rpy="0 0 0"/>
+    <origin xyz="-0.387737 -0.001226 -0.082264" rpy="0 0 0"/>
     <geometry>
       <mesh filename="file://$(find bal_robot_urdf_description)/meshes/realsence_1.stl" scale="0.001 0.001 0.001"/>
@@ -60,5 +60,5 @@
   </visual>
   <collision>
-    <origin xyz="-0.187737 -0.001226 -0.082264" rpy="0 0 0"/>
+    <origin xyz="-0.387737 -0.001226 -0.082264" rpy="0 0 0"/>
     <geometry>
       <mesh filename="file://$(find bal_robot_urdf_description)/meshes/realsence_1.stl" scale="0.001 0.001 0.001"/>
@@ -186,4 +186,5 @@
   </collision>
 </link>
+<link name="realsence_1_optical"> </link>
 <joint name="Rigid 2" type="fixed">
   <origin xyz="0.117737 0.001226 0.164764" rpy="0 0 0"/>
@@ -196,4 +197,9 @@
   <child link="realsence_1"/>
 </joint>
+<joint name="Rigid 3 optical" type="fixed">
+  <origin xyz="0.187737 0.001226 0.082264" rpy="${-pi/2} 0 ${-pi/2}"/>
+  <parent link="base_link"/>
+  <child link="realsence_1_optical"/>
+</joint>
 <joint name="Revolute 4" type="continuous">
   <origin xyz="0.107737 -0.108774 0.054764" rpy="0 0 0"/>
